File: parallel_trail.kicad_sch (KiCad schematic)
At the start: 47 parts, among them U1 TL074, U2 PT2257, U3 TL074, U4 X9C103, U5 X9C103

Commit message: all new
Parts:
- removed C8: 100nf, Capacitor_THT:C_Rect_L10.0mm_W4.0mm_P7.50mm_MKS4, symbol Device:C
- removed U2: PT2257, Package_DIP:DIP-8_W7.62mm_LongPads, symbol Audio:PT2257
- removed U4, U5: X9C103, Package_DIP:DIP-8_W7.62mm_LongPads, symbol Potentiometer_Digital:X9C10X
- added C20: 100nf, Capacitor_SMD:C_0805_2012Metric, symbol Device:C
- added C21, C22, C23, C24, C25, C26, C27, C28, C30, C31, C32, C33, C8: 10uF, Capacitor_SMD:C_Elec_4x5.4, symbol Device:C_Polarized_US
- added C29, C34: 150pf, Capacitor_SMD:C_0805_2012Metric, symbol Device:C
- added R24, R28, R29, R31: 10k, Resistor_SMD:R_0805_2012Metric, symbol Device:R
- added R25, R30: 4.7k, Resistor_SMD:R_0805_2012Metric, symbol Device:R
- added R26, R27: 1M, Resistor_SMD:R_0805_2012Metric, symbol Device:R
- added R32, R33, R34, R35, R36, R37: 100k, Resistor_SMD:R_0805_2012Metric, symbol Device:R
- added U6: PT2258, Package_SO:SOP-20_7.5x12.8mm_P1.27mm, symbol Driver_Motor:PT2258
- C1, C2: footprint Capacitor_THT:C_Rect_L10.0mm_W4.0mm_P7.50mm_MKS4 -> Capacitor_SMD:C_0805_2012Metric
- C10: value 47uf -> 10uF; footprint Capacitor_THT:CP_Radial_D8.0mm_P3.80mm -> Capacitor_SMD:C_Elec_4x5.4
- C11, C7: value 220N -> 220nF; footprint Capacitor_THT:C_Rect_L10.0mm_W4.0mm_P7.50mm_MKS4 -> Capacitor_SMD:C_0805_2012Metric
- C12, C13, C16, C17, C18, C19, C3, C4, C5, C6, C9: footprint Capacitor_THT:CP_Radial_D8.0mm_P3.80mm -> Capacitor_SMD:C_Elec_4x5.4
- C14, C15: footprint Capacitor_THT:C_Disc_D5.0mm_W2.5mm_P2.50mm -> Capacitor_SMD:C_0805_2012Metric
- R1, R10, R11, R12, R13, R16, R17, R18, R19, R2, R20, R21, R22, R23, R3, R4, R5, R6, R7, R8, R9: footprint Resistor_THT:R_Axial_DIN0207_L6.3mm_D2.5mm_P10.16mm_Horizontal -> Resistor_SMD:R_0805_2012Metric
- R14, R15: value 33k -> 4.7k; footprint Resistor_THT:R_Axial_DIN0207_L6.3mm_D2.5mm_P10.16mm_Horizontal -> Resistor_SMD:R_0805_2012Metric
- U1, U3: footprint Package_DIP:DIP-14_W7.62mm_LongPads -> Package_SO:SO-14_3.9x8.65mm_P1.27mm
Connections:
- net +9V: now also C20.2, C21.1, U6.16 (VCC), U6.17 (CODE1); no longer C10.1
- net GND: now also C20.1, C21.2, C22.2, R25.2, R26.1, R27.1, R30.2, R32.1, R33.1, R34.1, R35.1, R36.1, R37.1, U6.14 (GND), U6.4 (CODE2), U6.5 (DGND); no longer C10.2
- net SCL: now also U6.6 (SCL)
- net SDA: now also U6.7 (SDA)
- net output_buffer_out_left: now also C27.2, R37.2; no longer C16.2, R16.1
- net output_buffer_out_left_inverted: now also C28.2, R32.2; no longer C19.2, R23.1
- net output_buffer_out_right: now also C32.2, R33.2; no longer C17.2, R17.1
- net output_buffer_out_right_inverted: now also C33.2, R34.2; no longer C18.2, R22.1
- net at C3.1, C4.1, U1.1: now also C34.1, R31.1; no longer U1.2 (-)
- net at C14.2, R14.1, U3.9 (-): now also R28.2
- net at C14.1, C16.1, R19.1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: now also R28.1
- net at C6.1, U1.7: now also C29.1, R24.1; no longer U1.6 (-)
- net parallel_vol_2_in: now reaches C6.2
- net parallel_vol_2_in: now also C23.2, R26.2
- net parallel_vol_2_out: now reaches C5.1
- net parallel_vol_2_out: now also C8.2, R35.2
- net at C15.1, C17.1, R18.1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: now also R29.1
- net at C15.2, R15.1, U3.2 (-): now also R29.2
- net parallel_vol_1_in: now reaches C4.2
- net parallel_vol_1_in: now also C24.2, R27.2; no longer R5.2
- new net: C24.1, U6.2 (IN2)
- new net: C34.2, R30.1, R31.2, U1.2 (-)
- new net: C23.1, U6.1 (IN1)
- new net: C31.1, U6.10 (IN6)
- new net: C33.1, U6.11 (OUT6)
- new net: C32.1, U6.12 (OUT5)
- new net: C28.1, U6.13 (OUT4)
- new net: C22.1, U6.15 (REF)
- new net: C27.1, U6.18 (OUT3)
- new net: C10.1, U6.19 (OUT2)
- new net: C8.1, U6.20 (OUT1)
- new net: C25.1, U6.3 (IN3)
- new net: C26.1, U6.8 (IN4)
- new net: C30.1, U6.9 (IN5)
- new net: C29.2, R24.2, R25.1, U1.6 (-)
- new net buffer_left_vol_in: C16.2, C25.2, R16.1
- new net buffer_left_vol_in_inverted: C19.2, C26.2, R23.1
- new net buffer_right_vol_in: C17.2, C30.2, R17.1
- new net buffer_right_vol_in_inverted: C18.2, C31.2, R22.1
- new net parallel_vol_1_out: C10.2, R36.2, R5.2
- no-connect marks 2 -> 0
Other:
- note added: "+10dB"
- moved on the sheet: C5
